File: AnalogEVSE.kicad_pcb (KiCad board)
At the start: 2 copper layers, 84.7 x 66 mm, 72 parts, among them K1 Relay, P1 230V, P2 Relay 2, P3 Relay 1, P4 Pilot, P5 Status LEDs, P6 Rext, P7 Power, Q1 BC337, Q2 BC557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

Commit message: KiCAD 5, BOM
Other:
- board text added: "www.analogevse.xyz v2.0.0 01/2019"
- board text removed: "analogevse.xyz v2.0.0 12/2018"
Changed lines of the file:
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@@
-(kicad_pcb (version 4) (host pcbnew 4.0.2-stable)
+(kicad_pcb (version 20171130) (host pcbnew "(5.0.1-3-g963ef8bb5)")
   (general
-    (links 136)
-    (no_connects 0)
-    (area 100.229999 24.664999 193.995334 125.195001)
     (thickness 1.6)
     (drawings 11)
@@
     (pad_drill 0.8)
     (pad_to_mask_clearance 0)
+    (solder_mask_min_width 0.25)
     (aux_axis_origin 0 0)
-    (visible_elements FFFEFFED)
+    (visible_elements FFFCFFED)
     (pcbplotparams
       (layerselection 0x01060_80000000)
       (usegerberextensions true)
+      (usegerberattributes false)
+      (usegerberadvancedattributes false)
+      (creategerberjobfile false)
       (excludeedgelayer true)
       (linewidth 0.150000)
@@
       (hpglpennumber 1)
       (hpglpenspeed 20)
-      (hpglpendiameter 15)
-      (hpglpenoverlay 2)
+      (hpglpendiameter 15.000000)
       (psnegative false)
       (psa4output false)
@@
       (drillshape 0)
       (scaleselection 1)
-      (outputdirectory gerber))
+      (outputdirectory "gerber"))
   )
   (net 0 "")
@@
     (descr "Condensateur polarise")
     (tags CP)
-    (fp_text reference C1 (at 0 0 360) (layer F.SilkS)
+    (fp_text reference C1 (at 0 0) (layer F.SilkS)
       (effects (font (size 1.016 1.016) (thickness 0.2032)))
     )
@@
     (descr "Condensateur polarise")
     (tags CP)
-    (fp_text reference C4 (at 0 0 360) (layer F.SilkS)
+    (fp_text reference C4 (at 0 0) (layer F.SilkS)
       (effects (font (size 1.016 1.016) (thickness 0.2032)))
     )
@@
   (module mylib:Relay placed (layer F.Cu)
     (at 176.149 32.131 270)
-    (fp_text reference K1 (at 6.985 0 360) (layer F.SilkS)
+    (fp_text reference K1 (at 6.985 0) (layer F.SilkS)
       (effects (font (size 1.016 1.016) (thickness 0.2032)))
     )
@@
   (module mylib:Term-2pin (layer F.Cu)
     (at 111.125 60.706 270)
-    (fp_text reference P6 (at 0 1.778 360) (layer F.SilkS)
+    (fp_text reference P6 (at 0 1.778) (layer F.SilkS)
       (effects (font (size 1.016 1.016) (thickness 0.2032)))
     )
@@
     (descr "Transistor TO18")
     (tags TO18)
-    (fp_text reference U1 (at -1.778 1.397 360) (layer F.SilkS)
+    (fp_text reference U1 (at -1.778 1.397) (layer F.SilkS)
       (effects (font (size 1.016 1.016) (thickness 0.2032)))
     )
@@
     (descr "Diode 3 pas")
     (tags "DIODE DEV")
-    (fp_text reference D7 (at 2.032 -1.524 360) (layer F.SilkS)
+    (fp_text reference D7 (at 2.032 -1.524) (layer F.SilkS)
       (effects (font (size 1.016 1.016) (thickness 0.2032)))
     )
@@
     (descr "Diode 3 pas")
     (tags "DIODE DEV")
-    (fp_text reference D11 (at -1.778 -2.286 360) (layer F.SilkS)
+    (fp_text reference D11 (at -1.778 -2.286) (layer F.SilkS)
       (effects (font (size 1.016 1.016) (thickness 0.2032)))
     )
@@
     (descr "14 pins DIL package, elliptical pads")
     (tags DIL)
-    (fp_text reference U3 (at 2.667 -0.127 360) (layer F.SilkS)
+    (fp_text reference U3 (at 2.667 -0.127) (layer F.SilkS)
       (effects (font (size 1 1) (thickness 0.25)))
     )
@@
     (descr "14 pins DIL package, elliptical pads")
     (tags DIL)
-    (fp_text reference U5 (at -4.953 0 360) (layer F.SilkS)
+    (fp_text reference U5 (at -4.953 0) (layer F.SilkS)
       (effects (font (size 1 1) (thickness 0.25)))
     )
@@
   (gr_line (start 137.541 77.978) (end 137.668 77.978) (angle 90) (layer F.SilkS) (width 0.2))
   (gr_line (start 137.541 73.025) (end 137.541 77.978) (angle 90) (layer F.SilkS) (width 0.4))
-  (gr_text "analogevse.xyz\nv2.0.0 12/2018" (at 141.6304 44.1706) (layer B.Cu)
+  (gr_text "www.analogevse.xyz\nv2.0.0 01/2019" (at 141.6304 44.1706) (layer B.Cu)
     (effects (font (size 1.5 1.5) (thickness 0.3)) (justify mirror))
   )
