File: AnalogEVSE.sch (KiCad schematic (older format))
At the start: 64 parts, among them K1 Relay, P1 230V, P2 Relay 2, P3 Relay 1, P4 Pilot, P5 Status LEDs, P6 Rext, P7 Power, Q1 BC337, Q2 BC557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

Commit message: KiCAD 5, BOM
Parts:
- C1, C4, C6: symbol CP1-RESCUE-AnalogEVSE -> AnalogEVSE-rescue:CP1-RESCUE-AnalogEVSE
- C10, C11, C12, C13, C2, C3, C5, C7, C8, C9: symbol C-RESCUE-AnalogEVSE -> AnalogEVSE-rescue:C-RESCUE-AnalogEVSE
- D1, D10, D12, D2, D3, D6: symbol DIODE -> AnalogEVSE:DIODE
- D11, D7, D8, D9: symbol LED-RESCUE-AnalogEVSE -> AnalogEVSE-rescue:LED-RESCUE-AnalogEVSE
- D4, D5: symbol ZENER -> AnalogEVSE-rescue:ZENER
- F1: symbol FUSE -> AnalogEVSE:FUSE
- K1: symbol RELAY_2RT -> AnalogEVSE:RELAY_2RT
- P1, P3, P4, P6, P7: symbol CONN_2 -> AnalogEVSE:CONN_2
- P2, P5: symbol CONN_3 -> AnalogEVSE-rescue:CONN_3
- Q1, Q3: symbol NPN -> AnalogEVSE:NPN
- Q2: symbol PNP -> AnalogEVSE:PNP
- R1, R10, R11, R12, R13, R14, R15, R16, R17, R18, R19, R2, R3, R4, R5, R6, R7, R8, R9: symbol R-RESCUE-AnalogEVSE -> AnalogEVSE-rescue:R-RESCUE-AnalogEVSE
- RV1: symbol POT -> AnalogEVSE-rescue:POT
- T1: symbol TRANSFO -> AnalogEVSE:TRANSFO
- U1: symbol LM7812 -> AnalogEVSE:LM7812
- U2: symbol LM7912 -> AnalogEVSE:LM7912
- U3, U5: symbol LM339-RESCUE-AnalogEVSE -> AnalogEVSE-rescue:LM339-RESCUE-AnalogEVSE
- U4: symbol 4060 -> AnalogEVSE:4060
- Y1: symbol Crystal_Small -> Device:Crystal_Small
Connections:
- net +12V: no longer U3.3 (V+), U3.3 (V+), U3.3 (V+), U5.3 (V+), U5.3 (V+), U5.3 (V+)
- net -12V: no longer U3.12 (GND), U3.12 (GND), U3.12 (GND), U5.12 (GND), U5.12 (GND), U5.12 (GND)
