File: AnalogEVSE.sch (KiCad schematic (older format))
At the start: 64 parts, among them K1 Relay, P1 230V, P2 Relay 2, P3 Relay 1, P4 Pilot, P5 Status LEDs, P6 Rext, P7 Power, Q1 BC337, Q2 BC557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

Commit message: Cleanup
Parts:
- C3: value 220n -> 1u
Changed lines of the file:
@@
 Sheet 1 1
 Title "AnalogEVSE 2.0.0"
-Date "2018-07-21"
+Date "2019-01-03"
 Rev "2.0.0"
 Comp ""
@@
 P 5900 1200
 F 0 "C3" H 5900 1300 40  0000 L CNN
-F 1 "220n" H 5906 1115 40  0000 L CNN
+F 1 "1u" H 5906 1115 40  0000 L CNN
 F 2 "mylib:C2" H 5938 1050 30  0001 C CNN
 F 3 "~" H 5900 1200 60  0000 C CNN
